Commit message: add HOKUYO urg_node and slam toolbox to Dockerfile; update URDF to include laser frame and joint

File: src/epos4_controller/urdf/rerobot.urdf (robot description, URDF)
Before this commit: robot rerobot, 3 links, 2 joints
Links:
- added link laser_frame; visual cylinder length=0.04 radius=0.04
Joints:
- added joint laser_joint: type fixed, parent base_link, child laser_frame, origin xyz=0 0 0.714 rpy=0 0 0

Commit message: update README with hardware setup instructions; modify params.yaml for motor inversion; adjust URDF for laser frame naming; comment out unused robot_state_publisher node in launch file

File: src/epos4_controller/urdf/rerobot.urdf (robot description, URDF)
Before this commit: robot rerobot, 4 links, 3 joints
Links:
- removed link laser_frame
- added link laser; visual cylinder length=0.04 radius=0.04
Joints:
- joint laser_joint: child laser_frame -> laser
