Commit message: feat: update slam_toolbox configuration for improved map regeneration and scan matching thresholds

File: ros2_ws_main/src/bringup/rerobot_bringup/urdf/rerobot_2d.urdf (robot description, URDF)
Before this commit: robot rerobot, 4 links, 3 joints
Joints:
- joint laser_joint: origin xyz=0 0 0.714 rpy=0 0 0 -> xyz=0 0 0.714 rpy=3.141592653589793 0 0

Commit message: Add unit and integration tests for BNO086 IMU driver in advance

File: ros2_ws_main/src/bringup/rerobot_bringup/urdf/rerobot_2d.urdf (robot description, URDF)
Before this commit: robot rerobot, 4 links, 3 joints
Links:
- added link imu_link; visual box size=0.03 0.03 0.01
Joints:
- added joint imu_joint: type fixed, parent base_link, child imu_link, origin xyz=0 0 0.714 rpy=0 0 0

File: ros2_ws_main/src/bringup/rerobot_bringup/urdf/rerobot_3d.urdf (robot description, URDF)
Before this commit: robot rerobot, 4 links, 3 joints
Links:
- added link imu_link; visual box size=0.03 0.03 0.01
Joints:
- added joint imu_joint: type fixed, parent base_link, child imu_link, origin xyz=0 0 0.714 rpy=0 0 0
