Commit message: fix imu direction

File: ros2_ws_main/src/bringup/rerobot_bringup/urdf/rerobot.urdf (robot description, URDF)
Before this commit: robot rerobot, 6 links, 5 joints
Joints:
- joint imu_joint: origin xyz=0 0 0.64 rpy=0 0 1.5707963267948966 -> xyz=0 0 0.64 rpy=3.1415926535897932 0 1.5707963267948966

Commit message: feat: Implement EKF odometry with BNO086 IMU integration
- Added EKF odometry implementation in `epos4_odometry.cpp` to fuse wheel odometry and IMU data.
- Introduced new configuration files: `ekf.yaml` for EKF parameters and updated `params.yaml` for covariance settings.
- Modified launch files to support EKF integration, ensuring proper TF handling to avoid double publishing.
- Updated sensor configurations to reflect the new IMU setup and corrected URDF for accurate sensor orientation.
- Enhanced teleoperation node to warn users about missing parameter files affecting distance calculations.
- Documented the implementation walkthrough in `2026-08-11_ekf_odometry_code_walkthrough.md`.

File: ros2_ws_main/src/bringup/rerobot_bringup/urdf/rerobot.urdf (robot description, URDF)
Before this commit: robot rerobot, 6 links, 5 joints
Joints:
- joint imu_joint: origin xyz=0 0 0.64 rpy=3.1415926535897932 0 1.5707963267948966 -> xyz=0 0 0.64 rpy=0 0 1.5707963267948966
