Commit message: Add sensor configuration and URDF files for tilted and flat mounting presets
- Created a new sensor configuration file for tilted 45 degrees (config_sensors.tilted45.json) with detailed IMU and LiDAR settings.
- Added URDF files for flat (rerobot.flat.urdf) and tilted 15 degrees (rerobot.tilted15.urdf) configurations, integrating both 2D and 3D LiDARs along with the BNO086 IMU.
- Updated the existing tilted 45 degrees URDF (rerobot.tilted45.urdf) to reflect the new mounting configuration and sensor positions.
- Modified the main URDF file (rerobot.urdf) to include updated sensor positions and orientations based on recent measurements.

File: ros2_ws_main/src/bringup/rerobot_bringup/urdf/rerobot.flat.urdf (robot description, URDF)
Before this commit: robot rerobot, 6 links, 5 joints
Joints:
- joint rfans_joint: origin xyz=-0.02 0 0.75 rpy=0 -0.7853981634 3.1415926536 -> xyz=-0.075 0 0.725 rpy=0 0 0

File: ros2_ws_main/src/bringup/rerobot_bringup/urdf/rerobot.tilted15.urdf (robot description, URDF)
Before this commit: robot rerobot, 6 links, 5 joints
Joints:
- joint rfans_joint: origin xyz=-0.02 0 0.75 rpy=0 -0.7853981634 3.1415926536 -> xyz=-0.037 0 0.73 rpy=0 0.2617993878 0

Commit message: renew params for new body

File: ros2_ws_main/src/bringup/rerobot_bringup/urdf/rerobot.flat.urdf (robot description, URDF)
Before this commit: robot rerobot, 6 links, 5 joints
Links:
- link m1_wheel_link: geometry visual cylinder length=0.05 radius=0.128
- link m2_wheel_link: geometry visual cylinder length=0.05 radius=0.128
Joints:
- joint imu_joint: origin xyz=0 0 0.64 rpy=0 0 1.5707963267948966 -> xyz=0 0 0.74196 rpy=0 0 1.5707963267948966
- joint laser_joint: origin xyz=0.07 0 0.215 rpy=0 0 0 -> xyz=0.067 0 0.09406 rpy=3.141592653589793 0 0
- joint m1_wheel: origin xyz=0 0.205 0.075 rpy=0 0 0 -> xyz=0 0.2645 0.128 rpy=0 0 0
- joint m2_wheel: origin xyz=0 -0.205 0.075 rpy=0 0 0 -> xyz=0 -0.2645 0.128 rpy=0 0 0
- joint rfans_joint: origin xyz=-0.075 0 0.725 rpy=0 0 0 -> xyz=0 0 0.80246 rpy=0 0 0

File: ros2_ws_main/src/bringup/rerobot_bringup/urdf/rerobot.tilted15.urdf (robot description, URDF)
Before this commit: robot rerobot, 6 links, 5 joints
Links:
- link m1_wheel_link: geometry visual cylinder length=0.05 radius=0.128
- link m2_wheel_link: geometry visual cylinder length=0.05 radius=0.128
Joints:
- joint imu_joint: origin xyz=0 0 0.64 rpy=0 0 1.5707963267948966 -> xyz=0 0 0.74196 rpy=0 0 1.5707963267948966
- joint laser_joint: origin xyz=0.07 0 0.215 rpy=0 0 0 -> xyz=0.067 0 0.09406 rpy=3.141592653589793 0 0
- joint m1_wheel: origin xyz=0 0.205 0.075 rpy=0 0 0 -> xyz=0 0.2645 0.128 rpy=0 0 0
- joint m2_wheel: origin xyz=0 -0.205 0.075 rpy=0 0 0 -> xyz=0 -0.2645 0.128 rpy=0 0 0
- joint rfans_joint: origin xyz=-0.037 0 0.73 rpy=0 0.2617993878 0 -> xyz=0.038 0 0.80746 rpy=0 0.2617993878 0

File: ros2_ws_main/src/bringup/rerobot_bringup/urdf/rerobot.tilted45.urdf (robot description, URDF)
Before this commit: robot rerobot, 6 links, 5 joints
Links:
- link m1_wheel_link: geometry visual cylinder length=0.05 radius=0.128
- link m2_wheel_link: geometry visual cylinder length=0.05 radius=0.128
Joints:
- joint imu_joint: origin xyz=0 0 0.64 rpy=0 0 1.5707963267948966 -> xyz=0 0 0.74196 rpy=0 0 1.5707963267948966
- joint laser_joint: origin xyz=0.07 0 0.215 rpy=0 0 0 -> xyz=0.067 0 0.09406 rpy=3.141592653589793 0 0
- joint m1_wheel: origin xyz=0 0.205 0.075 rpy=0 0 0 -> xyz=0 0.2645 0.128 rpy=0 0 0
- joint m2_wheel: origin xyz=0 -0.205 0.075 rpy=0 0 0 -> xyz=0 -0.2645 0.128 rpy=0 0 0
- joint rfans_joint: origin xyz=-0.02 0 0.75 rpy=0 -0.7853981634 3.1415926536 -> xyz=0.055 0 0.82746 rpy=0 -0.7853981634 3.1415926536

File: ros2_ws_main/src/bringup/rerobot_bringup/urdf/rerobot.urdf (robot description, URDF)
Before this commit: robot rerobot, 6 links, 5 joints
Links:
- link m1_wheel_link: geometry visual cylinder length=0.05 radius=0.128
- link m2_wheel_link: geometry visual cylinder length=0.05 radius=0.128
Joints:
- joint imu_joint: origin xyz=0 0 0.64 rpy=0 0 1.5707963267948966 -> xyz=0 0 0.74196 rpy=0 0 1.5707963267948966
- joint laser_joint: origin xyz=0.07 0 0.215 rpy=0 0 0 -> xyz=0.067 0 0.09406 rpy=3.141592653589793 0 0
- joint m1_wheel: origin xyz=0 0.205 0.075 rpy=0 0 0 -> xyz=0 0.2645 0.128 rpy=0 0 0
- joint m2_wheel: origin xyz=0 -0.205 0.075 rpy=0 0 0 -> xyz=0 -0.2645 0.128 rpy=0 0 0
- joint rfans_joint: origin xyz=-0.02 0 0.75 rpy=0 -0.7853981634 3.1415926536 -> xyz=0 0 0.80246 rpy=0 0 0

Commit message: Update sensor configurations and BNO086 driver settings
- Adjusted T_lidar_imu parameters in config_sensors.json, config_sensors.tilted15.json, and config_sensors.tilted45.json based on recalculated values for BNO086.
- Introduced a new bno086.yaml configuration file to set auto_tare to off and adjusted other parameters for the BNO086 driver.
- Updated rerobot_bringup.launch.py to change the default IMU rate from 100 Hz to 200 Hz and included the new bno086.yaml parameters file.
- Modified URDF files (rerobot.flat.urdf, rerobot.tilted15.urdf, rerobot.tilted45.urdf) to reflect the corrected IMU mounting orientation and added a comparison IMU (imu_wit).
- Updated bringup scripts (bringup2d.sh, bringup3d.sh) to set the default IMU to true and changed the default IMU rate to 200 Hz.

File: ros2_ws_main/src/bringup/rerobot_bringup/urdf/rerobot.flat.urdf (robot description, URDF)
Before this commit: robot rerobot, 6 links, 5 joints
Links:
- added link imu_wit_link; visual box size=0.05 0.035 0.015
Joints:
- added joint imu_wit_joint: type fixed, parent base_link, child imu_wit_link, origin xyz=-0.065 0 0.57746 rpy=3.141592653589793 0 0
- joint imu_joint: origin xyz=0 0 0.74196 rpy=0 0 1.5707963267948966 -> xyz=0 0 0.74196 rpy=3.141592653589793 0 -1.625736

File: ros2_ws_main/src/bringup/rerobot_bringup/urdf/rerobot.tilted15.urdf (robot description, URDF)
Before this commit: robot rerobot, 6 links, 5 joints
Links:
- added link imu_wit_link; visual box size=0.05 0.035 0.015
Joints:
- added joint imu_wit_joint: type fixed, parent base_link, child imu_wit_link, origin xyz=-0.065 0 0.57746 rpy=3.141592653589793 0 0
- joint imu_joint: origin xyz=0 0 0.74196 rpy=0 0 1.5707963267948966 -> xyz=0 0 0.74196 rpy=3.141592653589793 0 -1.625736

File: ros2_ws_main/src/bringup/rerobot_bringup/urdf/rerobot.tilted45.urdf (robot description, URDF)
Before this commit: robot rerobot, 6 links, 5 joints
Links:
- added link imu_wit_link; visual box size=0.05 0.035 0.015
Joints:
- added joint imu_wit_joint: type fixed, parent base_link, child imu_wit_link, origin xyz=-0.065 0 0.57746 rpy=3.141592653589793 0 0
- joint imu_joint: origin xyz=0 0 0.74196 rpy=0 0 1.5707963267948966 -> xyz=0 0 0.74196 rpy=3.141592653589793 0 -1.625736

Commit message: fix TF position for new length alumi frame.

File: ros2_ws_main/src/bringup/rerobot_bringup/urdf/rerobot.flat.urdf (robot description, URDF)
Before this commit: robot rerobot, 7 links, 6 joints
Joints:
- joint imu_joint: origin xyz=0 0 0.74196 rpy=3.141592653589793 0 -1.625736 -> xyz=0 0 0.73346 rpy=3.141592653589793 0 -1.625736
- joint imu_wit_joint: origin xyz=-0.065 0 0.57746 rpy=3.141592653589793 0 0 -> xyz=-0.065 0 0.56896 rpy=3.141592653589793 0 0
- joint rfans_joint: origin xyz=0 0 0.80246 rpy=0 0 0 -> xyz=0 0 0.79396 rpy=0 0 0

File: ros2_ws_main/src/bringup/rerobot_bringup/urdf/rerobot.tilted15.urdf (robot description, URDF)
Before this commit: robot rerobot, 7 links, 6 joints
Joints:
- joint imu_joint: origin xyz=0 0 0.74196 rpy=3.141592653589793 0 -1.625736 -> xyz=0 0 0.73346 rpy=3.141592653589793 0 -1.625736
- joint imu_wit_joint: origin xyz=-0.065 0 0.57746 rpy=3.141592653589793 0 0 -> xyz=-0.065 0 0.56896 rpy=3.141592653589793 0 0
- joint rfans_joint: origin xyz=0.038 0 0.80746 rpy=0 0.2617993878 0 -> xyz=0.038 0 0.79896 rpy=0 0.2617993878 0

File: ros2_ws_main/src/bringup/rerobot_bringup/urdf/rerobot.tilted45.urdf (robot description, URDF)
Before this commit: robot rerobot, 7 links, 6 joints
Joints:
- joint imu_joint: origin xyz=0 0 0.74196 rpy=3.141592653589793 0 -1.625736 -> xyz=0 0 0.73346 rpy=3.141592653589793 0 -1.625736
- joint imu_wit_joint: origin xyz=-0.065 0 0.57746 rpy=3.141592653589793 0 0 -> xyz=-0.065 0 0.56896 rpy=3.141592653589793 0 0
- joint rfans_joint: origin xyz=0.055 0 0.82746 rpy=0 -0.7853981634 3.1415926536 -> xyz=0.055 0 0.81896 rpy=0 -0.7853981634 3.1415926536

Commit message: feat(amcl_compare): Add new tools for AMCL comparison and evaluation
- Introduced `checkpoint.py` for evaluating multiple replay bags against a reference pose, calculating error metrics and performing Fisher's exact test.
- Added `compare.py` to assess AMCL variants by comparing their poses and scans against the original bag's odometry and map data, generating detailed reports.
- Created `compare_scans.py` to validate the consistency of laser scans between original and replayed bags, measuring beam agreement.
- Implemented `initialpose_relay.py` to resend initial poses multiple times to ensure AMCL variants receive them correctly during replay.
- Developed `replay.sh` script to facilitate the playback of bags with AMCL variants, including logging and cleanup mechanisms.
- Defined `variants_repeat.yaml` and `variants_repeat6.yaml` for configuring AMCL variants with multiple copies to analyze loss frequency under different conditions.

File: ros2_ws_main/src/bringup/rerobot_bringup/urdf/rerobot.flat.urdf (robot description, URDF)
Before this commit: robot rerobot, 7 links, 6 joints
Joints:
- joint imu_wit_joint: origin xyz=-0.065 0 0.56896 rpy=3.141592653589793 0 0 -> xyz=-0.065 0 0.71896 rpy=3.141592653589793 0 0

File: ros2_ws_main/src/bringup/rerobot_bringup/urdf/rerobot.tilted15.urdf (robot description, URDF)
Before this commit: robot rerobot, 7 links, 6 joints
Joints:
- joint imu_wit_joint: origin xyz=-0.065 0 0.56896 rpy=3.141592653589793 0 0 -> xyz=-0.065 0 0.71896 rpy=3.141592653589793 0 0

File: ros2_ws_main/src/bringup/rerobot_bringup/urdf/rerobot.tilted45.urdf (robot description, URDF)
Before this commit: robot rerobot, 7 links, 6 joints
Joints:
- joint imu_wit_joint: origin xyz=-0.065 0 0.56896 rpy=3.141592653589793 0 0 -> xyz=-0.065 0 0.71896 rpy=3.141592653589793 0 0

Commit message: feat: Update AMCL and Nav2 parameters for improved localization and navigation
- Increased transform_tolerance in amcl.yaml from 1.0 to 8.0 to enhance TF validity during motion, preventing immediate goal failures due to TF expiration.
- Adjusted failure_tolerance in nav2_params.yaml to -1.0, allowing the robot to wait indefinitely when obstructed instead of failing the path.
- Extended movement_time_allowance in progress_checker to 3600.0 seconds to prevent premature failure during static waiting.
- Updated robot footprint in local and global costmaps to reflect actual dimensions, improving obstacle detection and navigation accuracy.
- Added inf_is_valid parameter to laser sources to ensure proper handling of invalid laser readings.
- Introduced auto_run.launch.py to streamline autonomous driving startup, consolidating launch processes and minimizing user input.
- Adjusted laser_joint orientation in URDF files to correct alignment issues observed in RViz, ensuring accurate sensor data representation.

File: ros2_ws_main/src/bringup/rerobot_bringup/urdf/rerobot.flat.urdf (robot description, URDF)
Before this commit: robot rerobot, 7 links, 6 joints
Joints:
- joint laser_joint: origin xyz=0.067 0 0.09406 rpy=3.141592653589793 0 0 -> xyz=0.067 0 0.09406 rpy=3.141592653589793 0 -0.08727

File: ros2_ws_main/src/bringup/rerobot_bringup/urdf/rerobot.tilted15.urdf (robot description, URDF)
Before this commit: robot rerobot, 7 links, 6 joints
Joints:
- joint laser_joint: origin xyz=0.067 0 0.09406 rpy=3.141592653589793 0 0 -> xyz=0.067 0 0.09406 rpy=3.141592653589793 0 -0.08727

File: ros2_ws_main/src/bringup/rerobot_bringup/urdf/rerobot.tilted45.urdf (robot description, URDF)
Before this commit: robot rerobot, 7 links, 6 joints
Joints:
- joint laser_joint: origin xyz=0.067 0 0.09406 rpy=3.141592653589793 0 0 -> xyz=0.067 0 0.09406 rpy=3.141592653589793 0 -0.08727

Commit message: feat: Update sensor calibration and visualization configurations
- Adjusted T_lidar_imu values in config_sensors.tilted45.json for improved sensor alignment.
- Modified nav2.rviz to enhance visualization of global and local costmaps, including adjustments to alpha values and enabling visibility.
- Updated URDF files (rerobot.flat.urdf, rerobot.tilted15.urdf, rerobot.tilted45.urdf) to reflect new yaw adjustments for R-Fans and laser joints, ensuring accurate sensor positioning.
- Added new scripts for R-Fans yaw calibration (rfans_yaw_calib.py) and GLIM transformation calculations (glim_t_lidar_imu.py) to facilitate sensor alignment and configuration updates.
- Enhanced documentation in README.md to provide clear instructions for using the new calibration tools and understanding the adjustments made.

File: ros2_ws_main/src/bringup/rerobot_bringup/urdf/rerobot.flat.urdf (robot description, URDF)
Before this commit: robot rerobot, 7 links, 6 joints
Joints:
- joint laser_joint: origin xyz=0.067 0 0.09406 rpy=3.141592653589793 0 -0.08727 -> xyz=0.067 0 0.09406 rpy=3.141592653589793 0 0.0100
- joint rfans_joint: origin xyz=0 0 0.79396 rpy=0 0 0 -> xyz=0 0 0.79396 rpy=0 0 0.098

File: ros2_ws_main/src/bringup/rerobot_bringup/urdf/rerobot.tilted15.urdf (robot description, URDF)
Before this commit: robot rerobot, 7 links, 6 joints
Joints:
- joint laser_joint: origin xyz=0.067 0 0.09406 rpy=3.141592653589793 0 -0.08727 -> xyz=0.067 0 0.09406 rpy=3.141592653589793 0 0.0100
- joint rfans_joint: origin xyz=0.038 0 0.79896 rpy=0 0.2617993878 0 -> xyz=0.038 0 0.79896 rpy=0.02621100498 0.2605139463 0.1014338006

File: ros2_ws_main/src/bringup/rerobot_bringup/urdf/rerobot.tilted45.urdf (robot description, URDF)
Before this commit: robot rerobot, 7 links, 6 joints
Joints:
- joint laser_joint: origin xyz=0.067 0 0.09406 rpy=3.141592653589793 0 -0.08727 -> xyz=0.067 0 0.09406 rpy=3.141592653589793 0 0.0100
- joint rfans_joint: origin xyz=0.055 0 0.81896 rpy=0 -0.7853981634 3.1415926536 -> xyz=0.055 0 0.81896 rpy=-0.09753276397 -0.7806114434 -3.003440027
